File: usb-serial.kicad_pcb (KiCad board)
At the start: 4 copper layers, 68.5 x 42 mm, 38 parts, among them J2 DB25_Plug, U10 TDR2-1222WI, U11 PEME2-5-D12-D, U12 MAX22246, U13 MAX22246, U3 USBLC6-2SC6, U6 Interface_USB_CP2102N-A01-GQF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, U7 SN75155, U8 SN75155, U9 LM1117DT-5.0

Commit message: Add resistor to fix serial break support
There must be pulldown resistor of 10k from TxD to GND on the CP2102 to
make serial break to work.

Also, updated to use KiCad 9.0 as PCB design tool.
Parts:
- added R1: 10k, Resistor_SMD:R_0402_1005Metric, F.Cu at (105.2, 66.7)
Routing:
- net ~{TXD}: track 8.44 -> 9.72 mm
- net GND: track 29.2 -> 30.0 mm
Other:
- board text added: "Isolated USB-RS232 Adapter By Anders Sandahl 2024-2026"
- board text removed: "Isolated USB-RS232 Adapter By Anders Sandahl 2024/2025"
